Commit message: upload

File: src/binpacking/models/colors.urdf.xacro (robot description, xacro)
@@ -14,4 +14,7 @@
     <color rgba="0.12941176470588237 0.7647058823529411 0.43529411764705883 1.0" />
   </material>
+  <material name="plum" >
+    <color rgba="0.76078431372 0.57647058823 0.55294117647 1.0" />
+  </material>
   <material name="almostblack" >
     <color rgba="0.027450980392156862 0.050980392156862744 0.050980392156862744 1.0" />
